File: EuroClack - Green_Screen_2350.kicad_sch (KiCad schematic)
At the start: 254 parts, among them J1 C2982548, J10 CV_OUT_4, J11 C7471773, J12 Pin Header, J13 CV_GATE_IN_4, J14 AUDIO_OUT_1, J15 AUDIO_IN_1, J16 USB_C_Receptacle_USB2.0_14P, J17 USB_HOST, J18 Eurorack 10 pin socket, J19 C7470101, J2 AUDIO_IN_2, J20 STEMMA_QT, J21 C2856837, J22 C2856837, J23 CV_GATE_IN3, J24 CV_GATE_IN_4, J25 SM03B-SRSS-TB, J26 CV_OUT_3, J27 CV_OUT_4, J28 C2881890, J29 C7470089, J3 CV_GATE_IN_1, J30 FFC, J4 CV_GATE_IN_2, J5 CV_GATE_IN3, J6 AUDIO_OUT_2, J7 CV_OUT_1, J8 CV_OUT_2, J9 CV_OUT_3, Q1 A3400A, Q2 A3401A, Q3 A3401A, Q4 A3400A, SW3 RotaryEncoder_Switch, SW4 RotaryEncoder_Switch, SW5 USER2, SW6 SW_Push, SW7 SW_Push, U1 RP2350_80QFN, U10 SPX3819M5-L-5-0, U11 TL072, U12 TPS54302, U13 TL072, U14 SPX3819M5-L-3-3, U15 SRAM, U16 SPX3819M5-L-3-3, U17 TL072, U18 SN74LVC1T45DCK, U19 LM393, U2 PCM5102, U20 TL072, U21 LM393, U22 SN74LVC1T45DCK, U23 TPS54302, U3 MCP4728, U4 W25Q128JVS, U5 PCM1808PWR, U6 TL072, U7 REF3033, U8 TL072, U9 SPX3819M5-L-3-3, Y1 ABM8-272-T3

Commit message: Updated pinouts to work better
Parts:
- removed C88: 10u, Clacktronics:C_0805_2012Metric, symbol Device:C
- added J31: SM03B-SRSS-TB, Connector_JST:JST_SH_BM03B-SRSS-TB_1x03-1MP_P1.00mm_Vertical, symbol Connector_Generic_MountingPin:Conn_01x03_MountingPin
- J16: value USB_C_Receptacle_USB2.0_14P -> C168704
- L3: footprint RP2350_80QFN_minimal:L_pol_2016 -> green_screen:L_pol_2016
- L4: footprint green_screen:IND-SMD_L10.4-W10.3 -> green_screen:IND-SMD_L5.4-W5.2
- SW1: footprint green_screen:KEY-SMD_4P-L6.0-W6.0-P3.90-LS9.0 -> green_screen:SW-TH_4P-L5.0-W5.0-P4.50-LS6.5
- U1: footprint RP2350_80QFN_minimal:RP2350-QFN-80-1EP_10x10_P0.4mm_EP3.4x3.4mm_ThermalVias -> green_screen:RP2350-QFN-80-1EP_10x10_P0.4mm_EP3.4x3.4mm_ThermalVias
Connections:
- net +12V: now also J21.25 (Pin_25); no longer J21.17 (Pin_17)
- net +5V: now also J21.17 (Pin_17); no longer J21.18 (Pin_18)
- net 12V_JACK: now also J22.16 (Pin_16); no longer J22.24 (Pin_24)
- net 5V_JACK: now also J22.24 (Pin_24); no longer J22.23 (Pin_23)
- net DISPLAY_BLK_JACK: now also J22.17 (Pin_17); no longer J22.16 (Pin_16)
- net DISPLAY_CS_JACK: now also J22.21 (Pin_21); no longer J22.20 (Pin_20)
- net DISPLAY_DC_JACK: now also J22.22 (Pin_22); no longer J22.21 (Pin_21)
- net DISPLAY_RES_JACK: now also J22.18 (Pin_18); no longer J22.17 (Pin_17)
- net DISPLAY_SCL_JACK: now also J22.20 (Pin_20); no longer J22.19 (Pin_19)
- net DISPLAY_SDA_JACK: now also J22.19 (Pin_19); no longer J22.18 (Pin_18)
- net GND: now also J21.18 (Pin_18), SW6.1, SW7.1, U2.12 (SCK), J31.2 (Pin_2), J31.MP (MountPin); no longer J21.19 (Pin_19)
- net GNDA_JACK: now also J10.S, J26.S, J27.S, J7.S, J8.S, J9.S
- net GND_JACK: now also J22.23 (Pin_23); no longer J10.S, J22.22 (Pin_22), J26.S, J27.S, J7.S, J8.S, J9.S, SW6.1, SW7.1
- net HSTX12_DC: now also J21.19 (Pin_19); no longer J21.20 (Pin_20)
- net HSTX13_CS: now also J21.20 (Pin_20); no longer J21.21 (Pin_21)
- net HSTX14_SCK: now also J21.21 (Pin_21); no longer J21.22 (Pin_22)
- net HSTX15_DIN: now also J21.22 (Pin_22); no longer J21.23 (Pin_23)
- net HSTX16_RST: now also J21.23 (Pin_23); no longer J21.24 (Pin_24)
- net HSTX17_BLK: now also J21.24 (Pin_24); no longer J21.25 (Pin_25)
- net I2S_ADC_BCK: now also U1.3 (GPIO6); no longer U1.9 (GPIO11)
- net I2S_ADC_DOUT: now also U1.6 (GPIO8); no longer U1.8 (GPIO10)
- net I2S_ADC_LRCK: now also U1.4 (GPIO7); no longer U1.6 (GPIO8)
- net I2S_ADC_SCKI: now also U1.21 (GPIO21); no longer U1.7 (GPIO9)
- net I2S_DAC_BCK: now also U1.78 (GPIO1); no longer U1.4 (GPIO7)
- net I2S_DAC_DIN: now also U1.80 (GPIO3); no longer U1.3 (GPIO6)
- net I2S_DAC_LRCK: now also U1.79 (GPIO2); no longer U1.1 (GPIO4)
- net STEMMA_SCL: now also U1.2 (GPIO5), J31.1 (Pin_1); no longer U1.21 (GPIO21)
- net STEMMA_SDA: now also U1.1 (GPIO4), J31.3 (Pin_3); no longer U1.20 (GPIO20)
- net USB_HOST_DM_MICRO: now also U1.7 (GPIO9); no longer U1.78 (GPIO1)
- net USB_HOST_DP_MICRO: now also U1.8 (GPIO10); no longer U1.79 (GPIO2)
- removed net I2S_DAC_SCK: U1.2 (GPIO5), U2.12 (SCK)
- no-connect marks 23 -> 22
Other:
- note added: "(UART1_RX)"
- note added: "(UART1_TX)"
- note added: "UART"

Commit message: Changes
Connections:
- net I2S_ADC_BCK: now also U1.7 (GPIO9); no longer U1.3 (GPIO6)
- net I2S_ADC_DOUT: now also U1.9 (GPIO11); no longer U1.6 (GPIO8)
- net I2S_ADC_LRCK: now also U1.8 (GPIO10); no longer U1.4 (GPIO7)
- net I2S_DAC_BCK: now also U1.3 (GPIO6); no longer U1.78 (GPIO1)
- net I2S_DAC_DIN: now also U1.6 (GPIO8); no longer U1.80 (GPIO3)
- net I2S_DAC_LRCK: no longer U1.79 (GPIO2)
- net USB_HOST_DM_MICRO: now also U1.78 (GPIO1); no longer U1.7 (GPIO9)
- net USB_HOST_DP_MICRO: now also U1.79 (GPIO2); no longer U1.8 (GPIO10)
- no-connect marks 22 -> 23
Changed lines of the file:
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@@
 	(text "I2C_0"
 		(exclude_from_sim no)
-		(at 487.426 278.384 0)
+		(at 485.648 240.284 0)
 		(effects
 			(font
@@
 	)
 	(no_connect
+		(at 516.89 236.22)
+	)
+	(no_connect
 		(at 596.9 241.3)
 	)
@@
 	(wire
 		(pts
-			(xy 501.65 231.14) (xy 523.24 231.14)
+			(xy 501.65 231.14) (xy 524.51 231.14)
 		)
 		(stroke
@@
 	)
 	(label "I2S_ADC_BCK"
-		(at 518.16 243.84 180)
+		(at 516.89 251.46 180)
 		(effects
 			(font
@@
 	)
 	(label "I2S_ADC_LRCK"
-		(at 518.16 246.38 180)
+		(at 516.89 254 180)
 		(effects
 			(font
@@
 	)
 	(label "I2S_ADC_DOUT"
-		(at 518.16 248.92 180)
+		(at 516.89 256.54 180)
 		(effects
 			(font
@@
 	)
 	(label "USB_HOST_DM_MICRO"
-		(at 524.51 251.46 180)
+		(at 524.51 231.14 180)
 		(effects
 			(font
@@
 	)
 	(label "I2S_DAC_LRCK"
-		(at 518.16 233.68 180)
+		(at 519.43 246.38 180)
 		(effects
 			(font
@@
 	)
 	(label "I2S_DAC_BCK"
-		(at 516.89 231.14 180)
+		(at 518.16 243.84 180)
 		(effects
 			(font
@@
 	)
 	(label "I2S_DAC_DIN"
-		(at 516.89 236.22 180)
+		(at 518.16 248.92 180)
 		(effects
 			(font
@@
 	)
 	(label "USB_HOST_DP_MICRO"
-		(at 524.51 254 180)
+		(at 524.51 233.68 180)
 		(effects
 			(font

Commit message: CHAGNES
Connections:
- net +3.3V: no longer JP1.1 (A), JP2.1 (A)
- net GND: now also JP1.1 (A), JP2.1 (A)
- net GNDA_JACK: no longer J10.S, J13.S, J14.S, J15.S, J2.S, J23.S, J24.S, J26.S, J27.S, J3.S, J4.S, J5.S, J6.S, J7.S, J8.S, R85.1, R86.1, R87.1, R88.1, R89.1, R90.1, R95.1, R96.1
- net GND_JACK: now also J10.S, J13.S, J14.S, J15.S, J2.S, J23.S, J24.S, J26.S, J27.S, J3.S, J4.S, J5.S, J6.S, J7.S, J8.S, R85.1, R86.1, R87.1, R88.1, R89.1, R90.1, R95.1, R96.1

Commit message: More changes
Parts:
- removed SW1: ~, green_screen:SW-TH_4P-L5.0-W5.0-P4.50-LS6.5, symbol Switch:SW_Push
- removed SW5: USER2, green_screen:SW-TH_4P-L5.0-W5.0-P4.50-LS6.5, symbol Switch:SW_Push
- added SW1, SW2: ~, EasyEDA_Lib:SW-TH_PS-8556DVA-6PN, symbol EasyEDA_Lib:PS-8556DVA-6PN
- J17: footprint green_screen:USB-A-SMD_AF180-13.1 -> green_screen:USB-A-TH_C42536
Connections:
- net GND_JACK: now also SW1.1, SW2.1
- net SW_USR1_JACK: now also SW1.2
- net SW_USR2_JACK: now also SW2.2
- no-connect marks 23 -> 29
Other:
- note added: "FUTURE DESIGN CHANGES ===================== Power down memory save circuit Reset and program as a single button?"
- note removed: "C2834937"
