File: EuroClack - Green_Screen_2350.kicad_sch (KiCad schematic)
At the start: 254 parts, among them J1 C2982548, J10 CV_OUT_4, J11 C7471773, J12 Pin Header, J13 CV_GATE_IN_4, J14 AUDIO_OUT_1, J15 AUDIO_IN_1, J16 C168704, J17 USB_HOST, J18 Eurorack 10 pin socket, J19 C7470101, J2 AUDIO_IN_2, J20 STEMMA_QT, J21 C2856837, J22 C2856837, J23 CV_GATE_IN3, J24 CV_GATE_IN_4, J25 SM03B-SRSS-TB, J26 CV_OUT_3, J27 CV_OUT_4, J28 C2881890, J29 C7470089, J3 CV_GATE_IN_1, J30 FFC, J31 SM03B-SRSS-TB, J4 CV_GATE_IN_2, J5 CV_GATE_IN3, J6 AUDIO_OUT_2, J7 CV_OUT_1, J8 CV_OUT_2, J9 CV_OUT_3, Q1 A3400A, Q2 A3401A, Q3 A3401A, Q4 A3400A, SW3 RotaryEncoder_Switch, SW4 RotaryEncoder_Switch, SW6 SW_Push, SW7 SW_Push, U1 RP2350_80QFN, U10 SPX3819M5-L-5-0, U11 TL072, U12 TPS54302, U13 TL072, U14 SPX3819M5-L-3-3, U15 SRAM, U16 SPX3819M5-L-3-3, U17 TL072, U18 SN74LVC1T45DCK, U19 LM393, U2 PCM5102, U20 TL072, U21 LM393, U22 SN74LVC1T45DCK, U23 TPS54302, U3 MCP4728, U4 W25Q128JVS, U5 PCM1808PWR, U6 TL072, U7 REF3033, U8 TL072, U9 SPX3819M5-L-3-3, Y1 ABM8-272-T3

Commit message: @@
Connections:
- net 12V_JACK: now also J22.25 (Pin_25); no longer J22.16 (Pin_16)
- net 5V_JACK: now also J22.17 (Pin_17); no longer J22.24 (Pin_24)
- net AUDIO_IN_1_JACK: now also J22.1 (Pin_1); no longer J22.40 (Pin_40)
- net AUDIO_IN_2_JACK: now also J22.2 (Pin_2); no longer J22.39 (Pin_39)
- net AUDIO_OUT_1_JACK: now also J22.3 (Pin_3); no longer J22.38 (Pin_38)
- net AUDIO_OUT_2_JACK: now also J22.4 (Pin_4); no longer J22.37 (Pin_37)
- net CV_GATE_IN_3_JACK: now also J22.5 (Pin_5); no longer J22.36 (Pin_36)
- net CV_GATE_IN_4_JACK: now also J22.6 (Pin_6); no longer J22.35 (Pin_35)
- net CV_IN_1_JACK: now also J22.15 (Pin_15); no longer J22.26 (Pin_26)
- net CV_IN_2_JACK: now also J22.16 (Pin_16); no longer J22.25 (Pin_25)
- net CV_OUT_1_JACK: now also J22.40 (Pin_40); no longer J22.1 (Pin_1)
- net CV_OUT_2_JACK: now also J22.37 (Pin_37); no longer J22.4 (Pin_4)
- net CV_OUT_3_JACK: now also J22.39 (Pin_39); no longer J22.2 (Pin_2)
- net CV_OUT_4_JACK: now also J22.38 (Pin_38); no longer J22.3 (Pin_3)
- net DISPLAY_BLK_JACK: now also J22.24 (Pin_24); no longer J22.17 (Pin_17)
- net DISPLAY_CS_JACK: now also J22.20 (Pin_20); no longer J22.21 (Pin_21)
- net DISPLAY_DC_JACK: now also J22.19 (Pin_19); no longer J22.22 (Pin_22)
- net DISPLAY_RES_JACK: now also J22.23 (Pin_23); no longer J22.18 (Pin_18)
- net DISPLAY_SCL_JACK: now also J22.21 (Pin_21); no longer J22.20 (Pin_20)
- net DISPLAY_SDA_JACK: now also J22.22 (Pin_22); no longer J22.19 (Pin_19)
- net ENC1_A_JACK: now also J22.31 (Pin_31); no longer J22.10 (Pin_10)
- net ENC1_B_JACK: now also J22.32 (Pin_32); no longer J22.9 (Pin_9)
- net ENC1_SW_JACK: now also J22.30 (Pin_30); no longer J22.11 (Pin_11)
- net ENC2_A_JACK: now also J22.34 (Pin_34); no longer J22.7 (Pin_7)
- net ENC2_B_JACK: now also J22.35 (Pin_35); no longer J22.6 (Pin_6)
- net ENC2_SW_JACK: now also J22.33 (Pin_33); no longer J22.8 (Pin_8)
- net GATE_IN_1_JACK: now also J22.7 (Pin_7); no longer J22.34 (Pin_34)
- net GATE_IN_2_JACK: now also J22.8 (Pin_8); no longer J22.33 (Pin_33)
- net GATE_OUT_1_JACK: now also J22.13 (Pin_13); no longer J22.28 (Pin_28)
- net GATE_OUT_2_JACK: now also J22.14 (Pin_14); no longer J22.27 (Pin_27)
- net GND_JACK: now also J22.18 (Pin_18); no longer J22.23 (Pin_23)
- net I2S_DAC_LRCK: now also U1.4 (GPIO7)
- net SW_RUN_JACK: now also J22.27 (Pin_27); no longer J22.14 (Pin_14)
- net SW_USR1_JACK: now also J22.28 (Pin_28); no longer J22.13 (Pin_13)
- net SW_USR2_JACK: now also J22.29 (Pin_29); no longer J22.12 (Pin_12)
- net USB_DM_JACK: now also J22.12 (Pin_12); no longer J22.29 (Pin_29)
- net USB_DP_JACK: now also J22.11 (Pin_11); no longer J22.30 (Pin_30)
- net USB_HOST_DM_JACK: now also J22.10 (Pin_10); no longer J22.31 (Pin_31)
- net USB_HOST_DP_JACK: now also J22.9 (Pin_9); no longer J22.32 (Pin_32)
- net ~{SW_MENU_BOOT_JACK}: now also J22.26 (Pin_26); no longer J22.15 (Pin_15)
- net ~{USBH_PWR_EN_JACK}: now also J22.36 (Pin_36); no longer J22.5 (Pin_5)
- no-connect marks 29 -> 31
Changed lines of the file:
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@@
 	)
 	(no_connect
+		(at 570.23 414.02)
+	)
+	(no_connect
 		(at 487.68 143.51)
 	)
@@
 	)
 	(no_connect
+		(at 519.43 279.4)
+	)
+	(no_connect
 		(at 104.14 535.94)
 	)
@@
 	(wire
 		(pts
-			(xy 501.65 246.38) (xy 518.16 246.38)
+			(xy 501.65 246.38) (xy 519.43 246.38)
 		)
 		(stroke
@@
 	(symbol
 		(lib_id "Connector_Generic:Conn_01x40")
-		(at 675.64 520.7 180)
+		(at 675.64 518.16 0)
+		(mirror y)
 		(unit 1)
 		(exclude_from_sim no)
@@
 		(dnp no)
 		(property "Reference" "J22"
-			(at 673.608 520.6422 0)
+			(at 673.608 518.2178 0)
 			(effects
 				(font
@@
 		)
 		(property "Value" "C2856837"
-			(at 673.608 518.2179 0)
+			(at 673.608 520.6421 0)
 			(effects
 				(font
@@
 		)
 		(property "Footprint" "green_screen:FPC-SMD_40P-P0.50_XUNPU_FPC-05FB-40PH20"
-			(at 675.64 520.7 0)
+			(at 675.64 518.16 0)
 			(effects
 				(font
@@
 		)
 		(property "Datasheet" "~"
-			(at 675.64 520.7 0)
+			(at 675.64 518.16 0)
 			(effects
 				(font
@@
 		)
 		(property "Description" "Generic connector, single row, 01x40, script generated (kicad-library-utils/schlib/autogen/connector/)"
-			(at 675.64 520.7 0)
+			(at 675.64 518.16 0)
 			(effects
 				(font

Commit message: Prototype pushed
Parts:
- added R4: 0R, Clacktronics:R_0402_1005Metric, symbol Device:R
- C11, C13, C15, C21, C23, C24, C34, C36, C4, C45, C53, C57, C58, C60, C89, C96, C98: value 10u -> 10uF
- C38, C87: footprint Capacitor_SMD:CP_Elec_4x5.4 -> Capacitor_SMD:CP_Elec_5x5.4
- C7, C8: value 10p -> 2n2
- J10, J27: value CV_OUT_4 -> Stereo Jack
- J11: value C7471773 -> C22438074
- J13, J24: value CV_GATE_IN_4 -> Stereo Jack
- J14: value AUDIO_OUT_1 -> Stereo Jack
- J15: value AUDIO_IN_1 -> Stereo Jack
- J19: value C7470101 -> C22438194
- J2: value AUDIO_IN_2 -> Stereo Jack
- J23, J5: value CV_GATE_IN3 -> Stereo Jack
- J26, J9: value CV_OUT_3 -> Stereo Jack
- J28: value C2881890 -> C22438074
- J29: value C7470089 -> C22438194
- J3: value CV_GATE_IN_1 -> Stereo Jack
- J4: value CV_GATE_IN_2 -> Stereo Jack
- J6: value AUDIO_OUT_2 -> Stereo Jack
- J7: value CV_OUT_1 -> Stereo Jack
- J8: value CV_OUT_2 -> Stereo Jack
- L2: value 3.3uH 5A 20mOhm -> 10uH 4A; footprint green_screen:IND-SMD_L5.4-W5.2 -> green_screen:FXL0630-100-M
- L4: value 6.8uH 5A 20mOhm -> 10uH 4A; footprint green_screen:IND-SMD_L5.4-W5.2 -> green_screen:FXL0630-100-M
- R1, R15, R16, R2: value R -> 1k
- U15: footprint Package_SO:SOIC-8_5.3x5.3mm_P1.27mm -> Package_SO:SOIC-8_3.9x4.9mm_P1.27mm
- U5: footprint Package_SO:TSSOP-14_4.4x3.6mm_P0.4mm -> Package_SO:TSSOP-14_4.4x5mm_P0.65mm
Connections:
- net GNDA_JACK is gone; now on net GND_JACK: J9.S
- net +5V: now also R4.1; no longer L2.2, R91.2
- net GND: no longer SW6.1, SW7.1
- net GND_JACK: now also SW6.1, SW7.1
- new net: L2.2, R4.2, R91.2
- no-connect marks 31 -> 40
Other:
- note added: "AUDIO IN 1"
- note added: "AUDIO IN 2"
- note added: "AUDIO_OUT_1"
- note added: "AUDIO_OUT_2"
- note added: "CV_GATE_IN_1"
- note added: "CV_GATE_IN_2"
- note added: "CV_GATE_IN_3"
- note added: "CV_GATE_IN_4"
- note added: "CV_OUT_1"
- note added: "CV_OUT_2"
- note added: "CV_OUT_3"
- note added: "CV_OUT_4"
- note added: "Errors List Opamps are not suitable for 12V C38, C87 wrong footprint C8, C2, C1, C7 wrong footprint"
- note added: "GATE_IN_1"
- note added: "GATE_IN_2"
- note added: "GATE_OUT_1"
- note added: "GATE_OUT_2"

Commit message: Errors list
Connections:
- net CV_OUT_2: now reaches FB9.1, R35.2, R56.2
- net CV_OUT_3: now reaches FB10.1, R38.2, R55.2
- net CV_IN_1: now reaches FB3.2, R31.1
- net CV_OUT_4: now reaches FB11.1, R41.2, R54.2
- net CV_OUT_1: now reaches FB8.1, R18.2, R57.2
Other:
- note added: "Errors List Opamps are not suitable for 12V C38, C87 wrong footprint C8, C2, C1, C7 wrong footprint SDA/SCL are the wrong way around on MCP4728 Pullup needed on PCM5102 xmute remove jumper on 5v CV inputs to micro have no protection low pass on CV ADC inputs for anti alizing TVS diodes on outputs"
- note added: "FUTURE DESIGN CHANGES ===================== Power down memory save circuit Move TFT SPI to a ribbon connector on brain PCB so it is as short as possible Put (both?) I2C to the 40 pin connector More test points move USB to more ergonomic place, perhaps might need more HP Bezel design for display delete serial, move qwiic down put vref on adc vdd input of 2350"
- note added: "Test List ========= PCM1808 input ranges of opamps speed of comparators SD card in SDIO and SPI mode Noise on analog inputs and outputs USB host"
- note removed: "Errors List Opamps are not suitable for 12V C38, C87 wrong footprint C8, C2, C1, C7 wrong footprint"
- note removed: "FUTURE DESIGN CHANGES ===================== Power down memory save circuit Reset and program as a single button?"
- moved on the sheet: FB2, FB3
Changed lines of the file:
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@@
 		)
 	)
-	(text "Errors List\n\nOpamps are not suitable for 12V\nC38, C87 wrong footprint\nC8, C2, C1, C7 wrong footprint"
+	(text "Errors List\n\nOpamps are not suitable for 12V\nC38, C87 wrong footprint\nC8, C2, C1, C7 wrong footprint\nSDA/SCL are the wrong way around on MCP4728\nPullup needed on PCM5102 xmute\nremove jumper on 5v\nCV inputs to micro have no protection\nlow pass on CV ADC inputs for anti alizing\nTVS diodes on outputs\n\n"
 		(exclude_from_sim no)
-		(at -68.834 353.06 0)
+		(at 781.812 126.746 0)
 		(effects
 			(font
@@
 		)
 	)
-	(text "FUTURE DESIGN CHANGES\n=====================\n\nPower down memory save circuit\nReset and program as a single button?"
+	(text "FUTURE DESIGN CHANGES\n=====================\n\nPower down memory save circuit\nMove TFT SPI to a ribbon connector on brain PCB so it is as short as possible\nPut (both?) I2C to the 40 pin connector\nMore test points\nmove USB to more ergonomic place, perhaps might need more HP\nBezel design for display\ndelete serial, move qwiic down\nput vref on adc vdd input of 2350\n"
 		(exclude_from_sim no)
 		(at 792.48 93.472 0)
@@
 	(text "2 audio inputs - ac coupled\n4 CV / gate hybrid inputs\n2 audio / CV outputs\n4 CV outputs\n2 encoders with buttons\n2 user buttons\nSD card reader\nUSB host port\nUSB input port for programming and PC connection\nFull colour 240x280 display over SPI/HTSC\n"
 		(exclude_from_sim no)
-		(at 165.608 102.362 0)
+		(at 193.548 102.362 0)
 		(effects
 			(font
@@
 		)
 	)
+	(text "Test List\n=========\nPCM1808 input\nranges of opamps\nspeed of comparators\nSD card in SDIO and SPI mode\nNoise on analog inputs and outputs\nUSB host"
+		(exclude_from_sim no)
+		(at 780.034 150.622 0)
+		(effects
+			(font
+				(size 1.27 1.27)
+			)
+		)
+	)
 	(junction
 		(at 552.45 462.28)
@@
 	(wire
 		(pts
-			(xy 171.45 294.64) (xy 172.72 294.64)
+			(xy 163.83 294.64) (xy 172.72 294.64)
 		)
 		(stroke
@@
 	(wire
 		(pts
-			(xy 142.24 332.74) (xy 165.1 332.74)
+			(xy 142.24 332.74) (xy 156.21 332.74)
 		)
 		(stroke
@@
 	(wire
 		(pts
-			(xy 140.97 294.64) (xy 166.37 294.64)
+			(xy 140.97 294.64) (xy 158.75 294.64)
 		)
 		(stroke
@@
 	(wire
 		(pts
-			(xy 170.18 332.74) (xy 172.72 332.74)
+			(xy 161.29 332.74) (xy 172.72 332.74)
 		)
 		(stroke
@@
 		)
 	)
+	(label "CV_OUT_4"
+		(at 701.04 363.22 180)
+		(effects
+			(font
+				(size 1.27 1.27)
+			)
+			(justify right bottom)
+		)
+	)
 	(label "USB_HOST_DM_MICRO"
 		(at 524.51 231.14 180)
@@
 		)
 	)
+	(label "CV_OUT_2"
+		(at 711.2 297.18 180)
+		(effects
+			(font
+				(size 1.27 1.27)
+			)
+			(justify right bottom)
+		)
+	)
 	(label "~{SW_MENU_BOOT_MICRO}"
 		(at 641.35 533.4 0)
@@
 		)
 	)
+	(label "CV_OUT_1"
+		(at 702.31 260.35 180)
+		(effects
+			(font
+				(size 1.27 1.27)
+			)
+			(justify right bottom)
+		)
+	)
 	(label "DISPLAY_SDA_JACK"
 		(at 502.92 125.73 0)
@@
 		)
 	)
+	(label "CV_IN_1"
+		(at 163.83 332.74 0)
+		(effects
+			(font
+				(size 1.27 1.27)
+			)
+			(justify left bottom)
+		)
+	)
 	(label "HSTX14_SCK"
 		(at 516.89 264.16 180)
@@
 		)
 	)
+	(label "CV_OUT_3"
+		(at 702.31 330.2 180)
+		(effects
+			(font
+				(size 1.27 1.27)
+			)
+			(justify right bottom)
+		)
+	)
 	(label "HSTX13_CS"
 		(at 645.16 518.16 0)
@@
 	(symbol
 		(lib_id "Device:FerriteBead_Small")
-		(at 167.64 332.74 90)
+		(at 158.75 332.74 90)
 		(unit 1)
 		(exclude_from_sim no)
@@
 		(fields_autoplaced yes)
 		(property "Reference" "FB3"
-			(at 167.6019 326.8937 90)
+			(at 158.7119 326.8937 90)
 			(effects
 				(font
@@
 		)
 		(property "Value" "F"
-			(at 167.6019 329.318 90)
+			(at 158.7119 329.318 90)
 			(effects
 				(font
@@
 		)
 		(property "Footprint" "Inductor_SMD:L_0402_1005Metric_Pad0.77x0.64mm_HandSolder"
-			(at 167.64 334.518 90)
+			(at 158.75 334.518 90)
 			(effects
 				(font
@@
 		)
 		(property "Datasheet" "~"
-			(at 167.64 332.74 0)
+			(at 158.75 332.74 0)
 			(effects
 				(font
@@
 		)
 		(property "Description" "Ferrite bead, small symbol"
-			(at 167.64 332.74 0)
+			(at 158.75 332.74 0)
 			(effects
 				(font
@@
 	(symbol
 		(lib_id "Device:FerriteBead_Small")
-		(at 168.91 294.64 90)
+		(at 161.29 294.64 90)
 		(unit 1)
 		(exclude_from_sim no)
@@
 		(fields_autoplaced yes)
 		(property "Reference" "FB2"
-			(at 168.8719 288.7937 90)
+			(at 161.2519 288.7937 90)
 			(effects
 				(font
@@
 		)
 		(property "Value" "F"
-			(at 168.8719 291.218 90)
+			(at 161.2519 291.218 90)
 			(effects
 				(font
@@
 		)
 		(property "Footprint" "Inductor_SMD:L_0402_1005Metric_Pad0.77x0.64mm_HandSolder"
-			(at 168.91 296.418 90)
+			(at 161.29 296.418 90)
 			(effects
 				(font
@@
 		)
 		(property "Datasheet" "~"
-			(at 168.91 294.64 0)
+			(at 161.29 294.64 0)
 			(effects
 				(font
@@
 		)
 		(property "Description" "Ferrite bead, small symbol"
-			(at 168.91 294.64 0)
+			(at 161.29 294.64 0)
 			(effects
 				(font
