File: EuroClack - Green_Screen_2350.kicad_sch (KiCad schematic)
At the start: 255 parts, among them J1 C2982548, J10 Stereo Jack, J11 C22438074, J12 Pin Header, J13 Stereo Jack, J14 Stereo Jack, J15 Stereo Jack, J16 C168704, J17 USB_HOST, J18 Eurorack 10 pin socket, J19 C22438194, J2 Stereo Jack, J20 STEMMA_QT, J21 C2856837, J22 C2856837, J23 Stereo Jack, J24 Stereo Jack, J25 SM03B-SRSS-TB, J26 Stereo Jack, J27 Stereo Jack, J28 C22438074, J29 C22438194, J3 Stereo Jack, J30 FFC, J31 SM03B-SRSS-TB, J4 Stereo Jack, J5 Stereo Jack, J6 Stereo Jack, J7 Stereo Jack, J8 Stereo Jack, J9 Stereo Jack, Q1 A3400A, Q2 A3401A, Q3 A3401A, Q4 A3400A, SW3 RotaryEncoder_Switch, SW4 RotaryEncoder_Switch, SW6 SW_Push, SW7 SW_Push, U1 RP2350_80QFN, U10 SPX3819M5-L-5-0, U11 TL072, U12 TPS54302, U13 TL072, U14 SPX3819M5-L-3-3, U15 SRAM, U16 SPX3819M5-L-3-3, U17 TL072, U18 SN74LVC1T45DCK, U19 LM393, U2 PCM5102, U20 TL072, U21 LM393, U22 SN74LVC1T45DCK, U23 TPS54302, U3 MCP4728, U4 W25Q128JVS, U5 PCM1808PWR, U6 TL072, U7 REF3033, U8 TL072, U9 SPX3819M5-L-3-3, Y1 ABM8-272-T3

Commit message: Major re-orgainisation and LLM design reveiw
Parts:
- removed R4: 0R, Clacktronics:R_0402_1005Metric, symbol Device:R
- C1, C12, C14, C16, C2, C22, C25, C26, C27, C28, C29, C30, C31, C32, C33, C37, C39, C40, C41, C42, C43, C44, C46, C47, C48, C49, C5, C50, C51, C52, C54, C56, C59, C61, C62, C63, C64, C65, C66, C67, C68, C69, C7, C70, C71, C72, C73, C74, C75, C76, C77, C78, C79, C8, C80, C81, C82, C83, C84, C85, C86, C90, C91, C92, C93, C94, C97: footprint Clacktronics:C_0402_1005Metric -> EuroClack:C_0402_1005Metric
- C10, C9: value 0R -> 1u; footprint Clacktronics:C_0402_1005Metric -> EuroClack:C_0402_1005Metric
- C11, C13, C15, C21, C23, C24, C3, C34, C36, C4, C45, C53, C57, C58, C6, C60, C89, C95, C96, C98: footprint Clacktronics:C_0805_2012Metric -> EuroClack:C_0805_2012Metric
- J1: footprint green_screen:TF-SMD_TF-123-ARP9H15 -> EuroClack:TF-SMD_TF-123-ARP9H15
- J10, J13, J14, J15, J2, J23, J24, J26, J27, J3, J4, J5, J6, J7, J8, J9: footprint green_screen:AUDIO-TH_PJ-301C -> EuroClack:AUDIO-TH_PJ-301C
- J11, J28: footprint green_screen:CONN-TH_8P-P1.27_DEALON_DW127R-11-08-34 -> EuroClack:CONN-TH_8P-P1.27_DEALON_DW127R-11-08-34
- J16: footprint green_screen:USB-C-TH_TYPE-C-USB-14P -> EuroClack:USB-C-TH_TYPE-C-USB-14P
- J17: footprint green_screen:USB-A-TH_C42536 -> EuroClack:USB-A-TH_C42536
- J19, J29: footprint green_screen:HDR-TH_8P-P1.27-H-M_1271WR-8P -> EuroClack:HDR-TH_8P-P1.27-H-M_1271WR-8P
- J21, J22: footprint green_screen:FPC-SMD_40P-P0.50_XUNPU_FPC-05FB-40PH20 -> EuroClack:FPC-SMD_40P-P0.50_XUNPU_FPC-05FB-40PH20
- J30: footprint green_screen:FPC-SMD_F1004-H-08-20G-R -> EuroClack:FPC-SMD_F1004-H-08-20G-R
- L2, L4: footprint green_screen:FXL0630-100-M -> EuroClack:FXL0630-100-M
- L3: footprint green_screen:L_pol_2016 -> EuroClack:L_pol_2016
- R1, R10, R100, R103, R104, R105, R106, R11, R12, R13, R14, R15, R16, R17, R18, R2, R22, R23, R24, R25, R26, R27, R28, R29, R3, R30, R31, R32, R33, R34, R35, R36, R37, R38, R39, R40, R41, R42, R43, R44, R45, R46, R47, R48, R49, R5, R50, R51, R52, R53, R54, R55, R56, R57, R6, R85, R86, R87, R88, R89, R9, R90, R92, R93, R94, R95, R96, R97, R98, R99: footprint Clacktronics:R_0402_1005Metric -> EuroClack:R_0402_1005Metric
- R101, R102: value ~ -> (none); footprint Clacktronics:R_0402_1005Metric -> EuroClack:R_0402_1005Metric
- R91: value 56K -> 75k; footprint Clacktronics:R_0402_1005Metric -> EuroClack:R_0402_1005Metric
- SW1, SW2: value ~ -> (none); footprint EasyEDA_Lib:SW-TH_PS-8556DVA-6PN -> EuroClack:SW-TH_PS-8556DVA-6PN; symbol EasyEDA_Lib:PS-8556DVA-6PN -> EuroClack:PS-8556DVA-6PN
- SW3, SW4: footprint green_screen:SW-TH_EC11XXXXXXXX -> EuroClack:SW-TH_EC11XXXXXXXX
- SW6, SW7: footprint green_screen:SW-TH_4P-L5.0-W5.0-P4.50-LS6.5 -> EuroClack:SW-TH_4P-L5.0-W5.0-P4.50-LS6.5
- U1: footprint green_screen:RP2350-QFN-80-1EP_10x10_P0.4mm_EP3.4x3.4mm_ThermalVias -> EuroClack:RP2350-QFN-80-1EP_10x10_P0.4mm_EP3.4x3.4mm_ThermalVias; symbol MCU_RaspberryPi_RP2350:RP2350_80QFN -> EuroClack:RP2350_80QFN
- U5: symbol PCM1808PWR:PCM1808PWR -> EuroClack:PCM1808PWR
Connections:
- net +12V: no longer U12.5 (EN)
- net +5V: now also L2.2, R91.2
- net 12V_JACK: no longer U23.5 (EN)
- no-connect marks 40 -> 42

Commit message: Further design review
Parts:
- added D3, D4: BAT54SW, Package_TO_SOT_SMD:SOT-323_SC-70, symbol Diode:BAT54SW
- R13, R26, R37, R40: value 20k -> 6.49k
- R17, R36, R39, R42: value 20k -> 1.96k
Connections:
- net I2S_DAC_MUTE is gone; now on net +3.3V: U2.17 (XSMT)
- net +5V: now also D3.2 (K), D4.2 (K)
- net GATE_IN_1_MICRO: now also D4.3 (COM)
- net GATE_IN_2_MICRO: now also D3.3 (COM)
- net GND: now also D3.1 (A), D4.1 (A)
- no-connect marks 42 -> 41
Other:
- note added: "U8 / U17: four calibrated +/-5V CV jack outputs U3 MCP4728: VDD=3.3VA; internal 2.048V reference, gain x1. Set VREF=1, G=0, PD=00 on all channels; save in EEPROM. Do not use gain x2 (4.096V exceeds the 3.3V supply). DAC inputs R17/R36/R39/R42 = 1.96k. Offset inputs R13/R26/R37/R40 = 6.49k. Feedback R18/R35/R38/R41 = 10k. Use 0.1% resistors for these networks and U11 R14/R25. U11 supplies VREF_ADC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"
- note removed: "VOUT = 0.000V to 4.096V * 4095/4096 for Gain of 2 Needs to be +-5V so 0-10V Gain of 10V / 4.096V = 2.44 10V / 2.44 = 4.098k nearest resistor 3.9k 10k / 3.9k = gain 2.56 4.094V = 10.49V Offset -5.25V from -3v 5.25V / 3.3V = 1.59 gain 10k / 1.59 = 6.29k nearest resistor two 3k3 in series 6.6k 10k / 6.8k = 1.52 gain offset -4.85V Output = 10.49 - 4.85 = +5.64V High -10.49 = -4.85V Low"

Commit message: Tweaks for next prototype
Parts:
- removed C36: 10uF, EuroClack:C_0805_2012Metric, symbol Device:C
- removed J12: Pin Header, Connector_PinHeader_2.54mm:PinHeader_1x08_P2.54mm_Vertical, symbol Connector_Generic:Conn_01x08
- removed J30: FFC, EuroClack:FPC-SMD_F1004-H-08-20G-R, symbol Connector_Generic:Conn_01x08
- added J12: Conn_01x16, symbol Connector_Generic:Conn_01x16
- added Q5: A3400A, Package_TO_SOT_SMD:SOT-23, symbol Device:Q_NMOS_GDS
- added R107: 10R, EuroClack:R_0402_1005Metric, symbol Device:R
- added R108: 100k, EuroClack:R_0402_1005Metric, symbol Device:R
Connections:
- net +12V: now also C85.2, U23.3 (VIN)
- net 12V_JACK: no longer C85.2, U23.3 (VIN)
- net 3V3_SD_SCREEN: now also J12.16 (Pin_16), J12.8 (Pin_8), J12.9 (Pin_9)
- net GND: now also C85.1, C87.2, C89.2, R98.1, U23.1 (GND), J12.10 (Pin_10), J12.11 (Pin_11), Q5.3 (S), R108.2
- net GND_JACK: no longer C85.1, C87.2, C89.2, R98.1, U23.1 (GND)
- net HSTX12_DC: now also J12.1 (Pin_1); no longer J21.19 (Pin_19)
- net HSTX13_CS: now also J12.2 (Pin_2); no longer J21.20 (Pin_20)
- net HSTX14_SCK: now also J12.3 (Pin_3); no longer J21.21 (Pin_21)
- net HSTX15_DIN: now also J12.4 (Pin_4); no longer J21.22 (Pin_22)
- net HSTX16_RST: now also J12.5 (Pin_5); no longer J21.23 (Pin_23)
- net HSTX17_BLK: now also R107.2, R108.1; no longer J21.24 (Pin_24)
- net I2C_DAC_SCL: now also J21.21 (Pin_21)
- net I2C_DAC_SDA: now also J21.22 (Pin_22)
- net STEMMA_SCL: now also J21.19 (Pin_19), J12.12 (Pin_12)
- net STEMMA_SDA: now also J21.20 (Pin_20), J12.13 (Pin_13)
- net DISPLAY_BLK_JACK: no longer names the net of J22.24 (Pin_24)
- net DISPLAY_CS_JACK: no longer names the net of J22.20 (Pin_20)
- net DISPLAY_DC_JACK: no longer names the net of J22.19 (Pin_19)
- net DISPLAY_RES_JACK: no longer names the net of J22.23 (Pin_23)
- net DISPLAY_SCL_JACK: no longer names the net of J22.21 (Pin_21)
- net DISPLAY_SDA_JACK: no longer names the net of J22.22 (Pin_22)
- new net: Q5.1 (G), R107.1
- new net LED_K: J12.6 (Pin_6), Q5.2 (D)
- new net SCREEN_TE: J12.7 (Pin_7)
- new net TP_INT: J12.15 (Pin_15)
- new net TP_RST: J12.14 (Pin_14)
Other:
- note added: "ASSOSIATION =========== HSTX13 HSTX15 NC HSTX 14 NC NC HSTX_16 HSTX_12 3V3 Screen GND 3v3 Screen Current limit + Transistor to HSTX17 STEMMA_SCL STEMMA_SDA GPIO 3 GPIO 20 TP_VCC"
- note added: "Errors List Opamps are not suitable for 12V C38, C87 wrong footprint C8, C2, C1, C7 wrong footprint SDA/SCL are the wrong way around on MCP4728 Jack sockets are connected wrong CV inputs to micro have no protection low pass on CV ADC inputs for anti alizing TVS diodes on outputs"
- note added: "FUTURE DESIGN CHANGES ===================== Power down memory save circuit Move TFT SPI to a ribbon connector on brain PCB so it is as short as possible Put (both?) I2C to the 40 pin connector More test points move USB to more ergonomic place, perhaps might need more HP Bezel design for display delete serial, move qwiic down"
- note added: "ON SCREEN ========= CS MOSI / QSPI D0 QSP1 D1 SCK QSPI_D3 QSPI_D2 RST (reset the screen) TE VDD GND LEDK LEDA TP_SCL TP_SDA TP_RST TP_INT TP_VCC"
- note added: "SCREEN"
- note added: "Test List ========= PCM1808 input ranges of opamps speed of comparators Noise on analog inputs and outputs USB host"
- note removed: "C2758340"
- note removed: "Errors List Opamps are not suitable for 12V C38, C87 wrong footprint C8, C2, C1, C7 wrong footprint SDA/SCL are the wrong way around on MCP4728 Pullup needed on PCM5102 xmute remove jumper on 5v CV inputs to micro have no protection low pass on CV ADC inputs for anti alizing TVS diodes on outputs"
- note removed: "FUTURE DESIGN CHANGES ===================== Power down memory save circuit Move TFT SPI to a ribbon connector on brain PCB so it is as short as possible Put (both?) I2C to the 40 pin connector More test points move USB to more ergonomic place, perhaps might need more HP Bezel design for display delete serial, move qwiic down put vref on adc vdd input of 2350"
- note removed: "Test List ========= PCM1808 input ranges of opamps speed of comparators SD card in SDIO and SPI mode Noise on analog inputs and outputs USB host"
- moved on the sheet: C85, C86, C87, C89, L4, R97, R98, U23

Commit message: Starting to re-arrange board
Parts:
- removed J31: SM03B-SRSS-TB, Connector_JST:JST_SH_BM03B-SRSS-TB_1x03-1MP_P1.00mm_Vertical, symbol Connector_Generic_MountingPin:Conn_01x03_MountingPin
- added D5, D6: BAT54SW, Package_TO_SOT_SMD:SOT-323_SC-70, symbol Diode:BAT54SW
- added J30: Conn_01x16, symbol Connector_Generic:Conn_01x16
- added J32: NV3030B QSPI, new_lcd:CONN-SMD_AXT524124, symbol Connector_Generic:Conn_02x12_Counter_Clockwise
- added J33: Conn_01x18, easyEDADownloader:FPC-SMD_18P-P0.50_FPC-0.5-18P-HYH2.0, symbol Connector_Generic:Conn_01x18
- added R58, R59, R60, R61: 1k, EuroClack:R_0402_1005Metric, symbol Device:R
- added U24: FM24CL16B, Package_SO:SOIC-8_3.9x4.9mm_P1.27mm, symbol Memory_NVRAM:FM24CL16B
- J12: footprint (none) -> Connector_FFC-FPC:Amphenol_F32Q-1A7x1-11016_1x16-1MP_P0.5mm_Horizontal
- J20: footprint Connector_JST:JST_SH_SM04B-SRSS-TB_1x04-1MP_P1.00mm_Horizontal -> Connector_JST:JST_SH_BM04B-SRSS-TB_1x04-1MP_P1.00mm_Vertical
- Q1, Q4, Q5: value A3400A -> AO3400A; symbol Device:Q_NMOS_GDS -> Transistor_FET:AO3400A
- Q2, Q3: value A3401A -> AO3401A; symbol Device:Q_PMOS_GDS -> Transistor_FET:AO3401A
Connections:
- net +12V: now also Q2.2 (S); no longer Q2.3 (S)
- net +3.3V: now also J32.15 (Pin_15), J32.17 (Pin_17), J32.23 (Pin_23), J33.17 (Pin_17), J33.3 (Pin_3), J33.4 (Pin_4), U24.8 (VDD)
- net +5V: now also D5.2 (K), D6.2 (K)
- net -12V: now also Q1.2 (S); no longer Q1.3 (S)
- net 3V3_SD_SCREEN: now also J30.16 (Pin_16), J30.8 (Pin_8), J30.9 (Pin_9)
- net 5V_JACK: now also Q3.2 (S); no longer Q3.3 (S)
- net GATE_IN_1_MICRO: now also R61.1; no longer D4.3 (COM), U21.3 (+)
- net GATE_IN_2_MICRO: now also R60.1; no longer D3.3 (COM), U21.5 (+)
- net GND: now also Q5.2 (S), D5.1 (A), D6.1 (A), J30.10 (Pin_10), J30.11 (Pin_11), J32.13 (Pin_13), J32.18 (Pin_18), J32.24 (Pin_24), J33.1 (Pin_1), J33.12 (Pin_12), J33.18 (Pin_18), J33.5 (Pin_5), J33.6 (Pin_6), U24.4 (VSS); no longer Q5.3 (S)
- net GND_JACK: now also Q4.2 (S); no longer Q4.3 (S)
- net HSTX12_DC: now also J30.1 (Pin_1)
- net HSTX13_CS: now also J30.2 (Pin_2)
- net HSTX14_SCK: now also J30.3 (Pin_3)
- net HSTX15_DIN: now also J30.4 (Pin_4)
- net HSTX16_RST: now also J30.5 (Pin_5)
- net LED_K: now also Q5.3 (D), J30.6 (Pin_6); no longer Q5.2 (D)
- net SCREEN_TE: now also J30.7 (Pin_7)
- net STEMMA_SCL: now also J30.12 (Pin_12), U24.6 (SCL)
- net STEMMA_SDA: now also J30.13 (Pin_13), U24.5 (SDA)
- net TP_INT: now also J30.15 (Pin_15), J32.22 (Pin_22), J33.16 (Pin_16)
- net TP_RST: now also J30.14 (Pin_14), J32.21 (Pin_21), J33.15 (Pin_15)
- net at FB12.2, R45.1: now also R58.1; no longer U19.3 (+)
- net at J18.1 (Pin_1), J18.2 (Pin_2): now also Q1.3 (D); no longer Q1.2 (D)
- net at FB5.2, R48.1: now also R59.1; no longer U19.5 (+)
- net at J18.10 (Pin_10), J18.9 (Pin_9): now also Q2.3 (D); no longer Q2.2 (D)
- net at Q3.1 (G), R99.1: now also Q4.3 (D); no longer Q4.2 (D)
- net at F1.1: now also Q3.3 (D); no longer Q3.2 (D)
- new net: D4.3 (COM), R61.2, U21.3 (+)
- new net: D6.3 (COM), R58.2, U19.3 (+)
- new net: D3.3 (COM), R60.2, U21.5 (+)
- new net: D5.3 (COM), R59.2, U19.5 (+)
- new net LCD_CS: J32.1 (Pin_1), J33.8 (Pin_8)
- new net LCD_DC: J33.7 (Pin_7)
- new net LCD_RST: J32.9 (Pin_9), J33.11 (Pin_11)
- new net LCD_TE: J32.14 (Pin_14)
- new net LEDK: J32.16 (Pin_16), J33.2 (Pin_2)
- new net QSPI_D1: J32.3 (Pin_3)
- new net QSPI_D2: J32.6 (Pin_6)
- new net QSPI_D3: J32.5 (Pin_5)
- new net SPI MOSI: J32.2 (Pin_2), J33.10 (Pin_10)
- new net SPI_SCK: J32.4 (Pin_4), J33.9 (Pin_9)
- new net TP_SCL: J32.19 (Pin_19), J33.13 (Pin_13)
- new net TP_SDA: J32.20 (Pin_20), J33.14 (Pin_14)
- no-connect marks 41 -> 47
Other:
- note added: "(ALSO QSPI0)"
- note added: "(also connected to logic)"
- note added: "Buydisplay ST7789"
- note added: "Non Voltatile RAM ================= ADC callibration DAC callibration"
- note added: "Non-Volatile Memory"
- note removed: "(UART1_RX)"
- note removed: "(UART1_TX)"
- note removed: "UART"
- moved on the sheet: D3, D4, J13, J15, J2, J23, J24, J3, J4, J5, R85, R86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
