File: EuroClack - Green_Screen_2350.kicad_pcb (KiCad board)
At the start: 4 copper layers, 109.2 x 110 mm, 269 parts, among them J1 C2982548, J10 CV_OUT_4, J11 C7471773, J12 Pin Header, J13 CV_GATE_IN_4, J14 AUDIO_OUT_1, J15 AUDIO_IN_1, J16 C168704, J17 USB_HOST, J18 Eurorack 10 pin socket, J19 C7470101, J2 AUDIO_IN_2, J20 STEMMA_QT, J21 C2856837, J22 C2856837, J23 CV_GATE_IN3, J24 CV_GATE_IN_4, J25 SM03B-SRSS-TB, J26 CV_OUT_3, J27 CV_OUT_4, J28 C2881890, J29 C7470089, J3 CV_GATE_IN_1, J30 FFC, J31 SM03B-SRSS-TB, J4 CV_GATE_IN_2, J5 CV_GATE_IN3, J6 AUDIO_OUT_2, J7 CV_OUT_1, J8 CV_OUT_2, J9 CV_OUT_3, Q1 A3400A, Q2 A3401A, Q3 A3401A, Q4 A3400A, SW3 RotaryEncoder_Switch, SW4 RotaryEncoder_Switch, SW6 SW_Push, SW7 SW_Push, U1 RP2350_80QFN, U10 SPX3819M5-L-5-0, U11 TL072, U12 TPS54302, U13 TL072, U14 SPX3819M5-L-3-3, U15 SRAM, U16 SPX3819M5-L-3-3, U17 TL072, U18 SN74LVC1T45DCK, U19 LM393, U2 PCM5102, U20 TL072, U21 LM393, U22 SN74LVC1T45DCK, U23 TPS54302, U3 MCP4728, U4 W25Q128JVS, U5 PCM1808PWR, U6 TL072, U7 REF3033, U8 TL072, U9 SPX3819M5-L-3-3, Y1 ABM8-272-T3

Commit message: @@
Parts:
- moved R89 23.5 mm to (106.8, 140.0), turned to 90 degrees
- moved R87 12.4 mm to (80.4, 140.7)
- moved J22 10.0 mm to (111.1, 81.0), turned to 180 degrees
- moved R85 9.01 mm to (80.5, 129.8), turned to 90 degrees
- moved R88 8.74 mm to (80.0, 152.5), turned to 90 degrees
- moved R90 7.68 mm to (106.9, 152.6), turned to 90 degrees
- moved R86 1.24 mm to (80.4, 116.2)
Connections:
- J22 pad 1: /CV_OUT_1_JACK -> /AUDIO_IN_1_JACK
- J22 pad 10: /ENC1_A_JACK -> /USB_HOST_DM_JACK
- J22 pad 11: /ENC1_SW_JACK -> /USB_DP_JACK
- J22 pad 12: /SW_USR2_JACK -> /USB_DM_JACK
- J22 pad 13: /SW_USR1_JACK -> /GATE_OUT_1_JACK
- J22 pad 14: /SW_RUN_JACK -> /GATE_OUT_2_JACK
- J22 pad 15: /~{SW_MENU_BOOT_JACK} -> /CV_IN_1_JACK
- J22 pad 16: /12V_JACK -> /CV_IN_2_JACK
- J22 pad 17: /DISPLAY_BLK_JACK -> /5V_JACK
- J22 pad 18: /DISPLAY_RES_JACK -> GND_JACK
- J22 pad 19: /DISPLAY_SDA_JACK -> /DISPLAY_DC_JACK
- J22 pad 2: /CV_OUT_3_JACK -> /AUDIO_IN_2_JACK
- J22 pad 20: /DISPLAY_SCL_JACK -> /DISPLAY_CS_JACK
- J22 pad 21: /DISPLAY_CS_JACK -> /DISPLAY_SCL_JACK
- J22 pad 22: /DISPLAY_DC_JACK -> /DISPLAY_SDA_JACK
- J22 pad 23: GND_JACK -> /DISPLAY_RES_JACK
- J22 pad 24: /5V_JACK -> /DISPLAY_BLK_JACK
- J22 pad 25: /CV_IN_2_JACK -> /12V_JACK
- J22 pad 26: /CV_IN_1_JACK -> /~{SW_MENU_BOOT_JACK}
- J22 pad 27: /GATE_OUT_2_JACK -> /SW_RUN_JACK
- J22 pad 28: /GATE_OUT_1_JACK -> /SW_USR1_JACK
- J22 pad 29: /USB_DM_JACK -> /SW_USR2_JACK
- J22 pad 3: /CV_OUT_4_JACK -> /AUDIO_OUT_1_JACK
- J22 pad 30: /USB_DP_JACK -> /ENC1_SW_JACK
- J22 pad 31: /USB_HOST_DM_JACK -> /ENC1_A_JACK
- J22 pad 32: /USB_HOST_DP_JACK -> /ENC1_B_JACK
- J22 pad 33: /GATE_IN_2_JACK -> /ENC2_SW_JACK
- J22 pad 34: /GATE_IN_1_JACK -> /ENC2_A_JACK
- J22 pad 35: /CV_GATE_IN_4_JACK -> /ENC2_B_JACK
- J22 pad 36: /CV_GATE_IN_3_JACK -> /~{USBH_PWR_EN_JACK}
- J22 pad 37: /AUDIO_OUT_2_JACK -> /CV_OUT_2_JACK
- J22 pad 38: /AUDIO_OUT_1_JACK -> /CV_OUT_4_JACK
- J22 pad 39: /AUDIO_IN_2_JACK -> /CV_OUT_3_JACK
- J22 pad 4: /CV_OUT_2_JACK -> /AUDIO_OUT_2_JACK
- J22 pad 40: /AUDIO_IN_1_JACK -> /CV_OUT_1_JACK
- J22 pad 5: /~{USBH_PWR_EN_JACK} -> /CV_GATE_IN_3_JACK
- J22 pad 6: /ENC2_B_JACK -> /CV_GATE_IN_4_JACK
- J22 pad 7: /ENC2_A_JACK -> /GATE_IN_1_JACK
- J22 pad 8: /ENC2_SW_JACK -> /GATE_IN_2_JACK
- J22 pad 9: /ENC1_B_JACK -> /USB_HOST_DP_JACK
- U1 pad 4: unconnected-(U1-GPIO7-Pad4) -> /I2S_DAC_LRCK
Routing:
- net /USB_DP_JACK: track 84.2 -> 1.29 mm, vias 2 -> 0
- net /CV_IN_1_JACK: track 0.00 -> 75.7 mm, vias 0 -> 1
- net /GATE_OUT_1_JACK: track 105.1 -> 45.9 mm, vias 2 -> 1
- net /GATE_IN_2_JACK: track 95.6 -> 51.4 mm
- net /ENC2_A_JACK: track 0.00 -> 43.4 mm, vias 0 -> 1
- net /GATE_IN_1_JACK: track 81.6 -> 39.1 mm
- net /CV_IN_2_JACK: track 127.4 -> 87.5 mm, vias 3 -> 1
- net /ENC2_SW_JACK: track 0.00 -> 35.3 mm, vias 0 -> 2
- net /ENC1_SW_JACK: track 44.1 -> 9.41 mm, vias 2 -> 1
- net /DISPLAY_RES_JACK: track 64.1 -> 29.7 mm, vias 4 -> 2
- net /AUDIO_OUT_1_JACK: track 81.3 -> 47.7 mm, vias 3 -> 1
- net /SW_USR1_JACK: track 34.1 -> 1.28 mm, vias 2 -> 1
- net /AUDIO_OUT_2_JACK: track 90.5 -> 59.7 mm, vias 3 -> 1
- net /DISPLAY_SDA_JACK: track 54.4 -> 29.4 mm, vias 4 -> 2
- net GND: track 149.4 -> 125.0 mm, vias 118 -> 116
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Other:
- outline, holes or cut-outs redrawn
- board text added: "AUDIO IN 1"
- board text added: "AUDIO IN 2"
- board text added: "AUDIO OUT 1"
- board text added: "AUDIO OUT 2"
- board text added: "CV IN 1"
- board text added: "CV IN 2"
- board text added: "CV OUT 1"
- board text added: "CV OUT 2"
- board text added: "CV OUT 3"
- board text added: "CV OUT 4"
- board text added: "CV/GATE IN 3"
- board text added: "CV/GATE IN 4"
- board text added: "DISPLAY"
- board text added: "ENCODER A"
- board text added: "ENCODER B"
- board text added: "GATE IN 1"
- board text added: "GATE IN 2"
- board text added: "GATE OUT 1"
- board text added: "GATE OUT 2"
- board text added: "SD"
- board text added: "USB HOST"

Commit message: Prototype pushed
Parts:
- added R4: 0R, Clacktronics:R_0402_1005Metric, F.Cu at (39.9, 63.9)
- added mouse-bite-2mm-slot: VAL**, green_screen:mouse-bite-2mm-slot, F.Cu at (33.6, 115.5)
- added mouse-bite-2mm-slot: VAL**, green_screen:mouse-bite-2mm-slot, F.Cu at (76.0, 61.9)
- added mouse-bite-2mm-slot: VAL**, green_screen:mouse-bite-2mm-slot, F.Cu at (76.0, 106.3)
- C11, C13, C15, C21, C23, C24, C34, C36, C4, C45, C53, C57, C58, C60, C89, C96, C98: value 10u -> 10uF
- C38, C87: footprint Capacitor_SMD:CP_Elec_4x5.4 -> Capacitor_SMD:CP_Elec_5x5.4
- C7, C8: value 10p -> 2n2
- J10, J27: value CV_OUT_4 -> Stereo Jack
- J11: value C7471773 -> C22438074
- J13, J24: value CV_GATE_IN_4 -> Stereo Jack
- J14: value AUDIO_OUT_1 -> Stereo Jack
- J15: value AUDIO_IN_1 -> Stereo Jack
- J19: value C7470101 -> C22438194
- J2: value AUDIO_IN_2 -> Stereo Jack
- J23, J5: value CV_GATE_IN3 -> Stereo Jack
- J26, J9: value CV_OUT_3 -> Stereo Jack
- J28: value C2881890 -> C22438074
- J29: value C7470089 -> C22438194
- J3: value CV_GATE_IN_1 -> Stereo Jack
- J4: value CV_GATE_IN_2 -> Stereo Jack
- J6: value AUDIO_OUT_2 -> Stereo Jack
- J7: value CV_OUT_1 -> Stereo Jack
- J8: value CV_OUT_2 -> Stereo Jack
- L2: value 3.3uH 5A 20mOhm -> 10uH 4A; footprint green_screen:IND-SMD_L5.4-W5.2 -> green_screen:FXL0630-100-M
- L4: value 6.8uH 5A 20mOhm -> 10uH 4A; footprint green_screen:IND-SMD_L5.4-W5.2 -> green_screen:FXL0630-100-M
- R1, R15, R16, R2: value R -> 1k
- U15: footprint Package_SO:SOIC-8_5.3x5.3mm_P1.27mm -> Package_SO:SOIC-8_3.9x4.9mm_P1.27mm
- U5: footprint Package_SO:TSSOP-14_4.4x3.6mm_P0.4mm -> Package_SO:TSSOP-14_4.4x5mm_P0.65mm
- moved R93 46.1 mm to (84.0, 93.4)
- moved R94 44.8 mm to (84.2, 89.5)
- moved JP1 7.83 mm to (72.9, 95.3), turned to 90 degrees
- moved R101 4.27 mm to (104.3, 107.0), turned to 0 degrees
- moved JP2 3.86 mm to (70.0, 95.3), turned to 90 degrees
- moved C87 3.17 mm to (126.1, 55.1)
- moved Q3 2.53 mm to (103.4, 104.5)
- moved C54 2.26 mm to (63.2, 80.1), turned to 180 degrees
- moved F1 2.20 mm to (100.3, 105.1)
- moved R12 2.19 mm to (72.2, 94.7), turned to 180 degrees
- moved J16 1.95 mm to (80.3, 91.5)
- moved C39 1.50 mm to (70.2, 93.6)
- moved C27 1.45 mm to (70.2, 94.7)
- moved C47 1.36 mm to (43.5, 73.2), turned to -90 degrees
- moved U6 1.25 mm to (66.0, 95.0)
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Connections:
- J9 pad S: /GNDA_JACK -> GND_JACK
- L2 pad 2: +5V -> Net-(L2-Pad2)
- R91 pad 2: +5V -> Net-(L2-Pad2)
- SW6 pad 1: GND -> GND_JACK
- SW7 pad 1: GND -> GND_JACK
Routing:
- net /SW_USR1_JACK: track 1.28 -> 47.7 mm
- net /5V_JACK: track 0.00 -> 41.9 mm, vias 0 -> 4
- net /SW_USR2_JACK: track 1.49 -> 36.7 mm, vias 1 -> 2
- net /DISPLAY_CS_JACK: track 25.9 -> 58.1 mm, vias 1 -> 2
- net /I2S_ADC_BCK: track 1.27 -> 33.4 mm, vias 1 -> 2
- net /DISPLAY_BLK_JACK: track 29.9 -> 61.7 mm, vias 1 -> 2
- net /USB_DM_JACK: track 1.29 -> 32.8 mm, vias 0 -> 1
- net /USB_DP_JACK: track 1.29 -> 32.4 mm, vias 0 -> 1
- net /~{SW_MENU_BOOT_JACK}: track 1.42 -> 31.6 mm
- net /DISPLAY_DC_JACK: track 25.4 -> 53.9 mm, vias 1 -> 2
- net /3V3_SD_SCREEN: track 39.2 -> 64.2 mm
- net /DISPLAY_RES_JACK: track 29.7 -> 53.5 mm
- net /DISPLAY_SDA_JACK: track 29.4 -> 51.3 mm
- net /DISPLAY_SCL_JACK: track 29.4 -> 49.1 mm
- net Net-(L2-Pad2): track 0.00 -> 16.0 mm
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- added copper zone on F.Cu, net /3V3_DAC
Other:
- outline, holes or cut-outs redrawn
- board text added: "CV-GATE IN 3"
- board text added: "CV-GATE IN 4"
- board text added: "GREENSCREEN 2350 PROTO 1"
- board text added: "MD0"
- board text added: "MD1"
- board text added: "QWIIC"
- board text added: "USB"
- board text removed: "CV/GATE IN 3"
- board text removed: "CV/GATE IN 4"
- board text removed: "STEMMAQT"
