File: EuroClack - Green_Screen_2350.kicad_pcb (KiCad board)
At the start: 4 copper layers, 109.2 x 110 mm, 273 parts, among them J1 C2982548, J10 Stereo Jack, J11 C22438074, J12 Pin Header, J13 Stereo Jack, J14 Stereo Jack, J15 Stereo Jack, J16 C168704, J17 USB_HOST, J18 Eurorack 10 pin socket, J19 C22438194, J2 Stereo Jack, J20 STEMMA_QT, J21 C2856837, J22 C2856837, J23 Stereo Jack, J24 Stereo Jack, J25 SM03B-SRSS-TB, J26 Stereo Jack, J27 Stereo Jack, J28 C22438074, J29 C22438194, J3 Stereo Jack, J30 FFC, J31 SM03B-SRSS-TB, J4 Stereo Jack, J5 Stereo Jack, J6 Stereo Jack, J7 Stereo Jack, J8 Stereo Jack, J9 Stereo Jack, Q1 A3400A, Q2 A3401A, Q3 A3401A, Q4 A3400A, SW3 RotaryEncoder_Switch, SW4 RotaryEncoder_Switch, SW6 SW_Push, SW7 SW_Push, U1 RP2350_80QFN, U10 SPX3819M5-L-5-0, U11 TL072, U12 TPS54302, U13 TL072, U14 SPX3819M5-L-3-3, U15 SRAM, U16 SPX3819M5-L-3-3, U17 TL072, U18 SN74LVC1T45DCK, U19 LM393, U2 PCM5102, U20 TL072, U21 LM393, U22 SN74LVC1T45DCK, U23 TPS54302, U3 MCP4728, U4 W25Q128JVS, U5 PCM1808PWR, U6 TL072, U7 REF3033, U8 TL072, U9 SPX3819M5-L-3-3, Y1 ABM8-272-T3

Commit message: Major re-orgainisation and LLM design reveiw
Parts:
- C1, C10, C12, C14, C16, C2, C22, C25, C26, C27, C28, C29, C30, C31, C32, C33, C37, C39, C40, C41, C42, C43, C44, C46, C47, C48, C49, C5, C50, C51, C52, C54, C56, C59, C61, C62, C63, C64, C65, C66, C67, C68, C69, C7, C70, C71, C72, C73, C74, C75, C76, C77, C78, C79, C8, C80, C81, C82, C83, C84, C85, C86, C9, C90, C91, C92, C93, C94, C97: footprint Clacktronics:C_0402_1005Metric -> EuroClack:C_0402_1005Metric
- C11, C13, C15, C21, C23, C24, C3, C34, C36, C4, C45, C53, C57, C58, C6, C60, C89, C95, C96, C98: footprint Clacktronics:C_0805_2012Metric -> EuroClack:C_0805_2012Metric
- J1: footprint green_screen:TF-SMD_TF-123-ARP9H15 -> EuroClack:TF-SMD_TF-123-ARP9H15
- J10, J13, J14, J15, J2, J23, J24, J26, J27, J3, J4, J5, J6, J7, J8, J9: footprint green_screen:AUDIO-TH_PJ-301C -> EuroClack:AUDIO-TH_PJ-301C
- J11, J28: footprint green_screen:CONN-TH_8P-P1.27_DEALON_DW127R-11-08-34 -> EuroClack:CONN-TH_8P-P1.27_DEALON_DW127R-11-08-34
- J16: footprint green_screen:USB-C-TH_TYPE-C-USB-14P -> EuroClack:USB-C-TH_TYPE-C-USB-14P
- J17: footprint green_screen:USB-A-TH_C42536 -> EuroClack:USB-A-TH_C42536
- J19, J29: footprint green_screen:HDR-TH_8P-P1.27-H-M_1271WR-8P -> EuroClack:HDR-TH_8P-P1.27-H-M_1271WR-8P
- J21, J22: footprint green_screen:FPC-SMD_40P-P0.50_XUNPU_FPC-05FB-40PH20 -> EuroClack:FPC-SMD_40P-P0.50_XUNPU_FPC-05FB-40PH20
- J30: footprint green_screen:FPC-SMD_F1004-H-08-20G-R -> EuroClack:FPC-SMD_F1004-H-08-20G-R
- L2, L4: footprint green_screen:FXL0630-100-M -> EuroClack:FXL0630-100-M
- L3: footprint RP2350_80QFN_minimal:L_pol_2016 -> EuroClack:L_pol_2016
- R1, R10, R100, R101, R102, R103, R104, R105, R106, R11, R12, R13, R14, R15, R16, R17, R18, R2, R22, R23, R24, R25, R26, R27, R28, R29, R3, R30, R31, R32, R33, R34, R35, R36, R37, R38, R39, R4, R40, R41, R42, R43, R44, R45, R46, R47, R48, R49, R5, R50, R51, R52, R53, R54, R55, R56, R57, R6, R85, R86, R87, R88, R89, R9, R90, R91, R92, R93, R94, R95, R96, R97, R98, R99: footprint Clacktronics:R_0402_1005Metric -> EuroClack:R_0402_1005Metric
- SW1, SW2: footprint EasyEDA_Lib:SW-TH_PS-8556DVA-6PN -> EuroClack:SW-TH_PS-8556DVA-6PN
- SW3, SW4: footprint green_screen:SW-TH_EC11XXXXXXXX -> EuroClack:SW-TH_EC11XXXXXXXX
- SW6, SW7: footprint green_screen:SW-TH_4P-L5.0-W5.0-P4.50-LS6.5 -> EuroClack:SW-TH_4P-L5.0-W5.0-P4.50-LS6.5
- U1: footprint RP2350_80QFN_minimal:RP2350-QFN-80-1EP_10x10_P0.4mm_EP3.4x3.4mm_ThermalVias -> EuroClack:RP2350-QFN-80-1EP_10x10_P0.4mm_EP3.4x3.4mm_ThermalVias
- mouse-bite-2mm-slot (x3): footprint green_screen:mouse-bite-2mm-slot -> EuroClack:mouse-bite-2mm-slot
